File: sirvo.v3.0.sch (EAGLE design)
At the start: 33 parts

Commit message: Finished routing of all on-board signals
Header routing not yet completed
Parts:
- removed JP2, JP4: M01SMD-4.5X1.5, SparkFun-Connectors:M01SMD-4.5X1.5
- added JP5, JP6: M01SMD-4.5X1.5, SparkFun-Connectors:M01SMD-4.5X1.5
Connections:
- net MOTOR_A: no longer JP1.1, JP3.1
- net MOTOR_B: no longer JP2.1, JP4.1
Other:
- moved on the sheet: JP1, JP3
Changed lines of the file:
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@@
 <grid distance="0.1" unitdist="inch" unit="inch" style="lines" multiple="1" display="no" altdistance="0.01" altunitdist="inch" altunit="inch"/>
 <layers>
-<layer number="1" name="Top" color="4" fill="1" visible="no" active="no"/>
-<layer number="16" name="Bottom" color="1" fill="1" visible="no" active="no"/>
-<layer number="17" name="Pads" color="2" fill="1" visible="no" active="no"/>
-<layer number="18" name="Vias" color="2" fill="1" visible="no" active="no"/>
-<layer number="19" name="Unrouted" color="6" fill="1" visible="no" active="no"/>
-<layer number="20" name="Dimension" color="15" fill="1" visible="no" active="no"/>
-<layer number="21" name="tPlace" color="16" fill="1" visible="no" active="no"/>
-<layer number="22" name="bPlace" color="14" fill="1" visible="no" active="no"/>
-<layer number="23" name="tOrigins" color="15" fill="1" visible="no" active="no"/>
-<layer number="24" name="bOrigins" color="15" fill="1" visible="no" active="no"/>
-<layer number="25" name="tNames" color="7" fill="1" visible="no" active="no"/>
-<layer number="26" name="bNames" color="7" fill="1" visible="no" active="no"/>
-<layer number="27" name="tValues" color="7" fill="1" visible="no" active="no"/>
-<layer number="28" name="bValues" color="7" fill="1" visible="no" active="no"/>
+<layer number="1" name="Top" color="4" fill="10" visible="yes" active="no"/>
+<layer number="16" name="Bottom" color="1" fill="1" visible="yes" active="no"/>
+<layer number="17" name="Pads" color="2" fill="1" visible="yes" active="no"/>
+<layer number="18" name="Vias" color="2" fill="1" visible="yes" active="no"/>
+<layer number="19" name="Unrouted" color="6" fill="1" visible="yes" active="no"/>
+<layer number="20" name="Dimension" color="15" fill="1" visible="yes" active="no"/>
+<layer number="21" name="tPlace" color="16" fill="1" visible="yes" active="no"/>
+<layer number="22" name="bPlace" color="14" fill="1" visible="yes" active="no"/>
+<layer number="23" name="tOrigins" color="15" fill="1" visible="yes" active="no"/>
+<layer number="24" name="bOrigins" color="15" fill="1" visible="yes" active="no"/>
+<layer number="25" name="tNames" color="7" fill="1" visible="yes" active="no"/>
+<layer number="26" name="bNames" color="7" fill="1" visible="yes" active="no"/>
+<layer number="27" name="tValues" color="7" fill="1" visible="yes" active="no"/>
+<layer number="28" name="bValues" color="7" fill="1" visible="yes" active="no"/>
 <layer number="29" name="tStop" color="7" fill="3" visible="no" active="no"/>
 <layer number="30" name="bStop" color="7" fill="6" visible="no" active="no"/>
@@
 <layer number="35" name="tGlue" color="7" fill="4" visible="no" active="no"/>
 <layer number="36" name="bGlue" color="7" fill="5" visible="no" active="no"/>
-<layer number="37" name="tTest" color="7" fill="1" visible="no" active="no"/>
-<layer number="38" name="bTest" color="7" fill="1" visible="no" active="no"/>
+<layer number="37" name="tTest" color="7" fill="1" visible="yes" active="no"/>
+<layer number="38" name="bTest" color="7" fill="1" visible="yes" active="no"/>
 <layer number="39" name="tKeepout" color="4" fill="11" visible="no" active="no"/>
 <layer number="40" name="bKeepout" color="1" fill="11" visible="no" active="no"/>
@@
 <layer number="44" name="Drills" color="7" fill="1" visible="no" active="no"/>
 <layer number="45" name="Holes" color="7" fill="1" visible="no" active="no"/>
-<layer number="46" name="Milling" color="3" fill="1" visible="no" active="no"/>
-<layer number="47" name="Measures" color="7" fill="1" visible="no" active="no"/>
-<layer number="48" name="Document" color="7" fill="1" visible="no" active="no"/>
-<layer number="49" name="Reference" color="7" fill="1" visible="no" active="no"/>
-<layer number="50" name="dxf" color="7" fill="1" visible="no" active="no"/>
-<layer number="51" name="tDocu" color="6" fill="1" visible="no" active="no"/>
-<layer number="52" name="bDocu" color="7" fill="1" visible="no" active="no"/>
-<layer number="53" name="tGND_GNDA" color="7" fill="9" visible="no" active="no"/>
-<layer number="54" name="bGND_GNDA" color="1" fill="9" visible="no" active="no"/>
-<layer number="56" name="wert" color="7" fill="1" visible="no" active="no"/>
-<layer number="57" name="tCAD" color="7" fill="1" visible="no" active="no"/>
+<layer number="46" name="Milling" color="3" fill="1" visible="yes" active="no"/>
+<layer number="47" name="Measures" color="7" fill="1" visible="yes" active="no"/>
+<layer number="48" name="Document" color="7" fill="1" visible="yes" active="no"/>
+<layer number="49" name="Reference" color="7" fill="1" visible="yes" active="no"/>
+<layer number="50" name="dxf" color="7" fill="1" visible="yes" active="no"/>
+<layer number="51" name="tDocu" color="6" fill="1" visible="yes" active="no"/>
+<layer number="52" name="bDocu" color="7" fill="1" visible="yes" active="no"/>
+<layer number="53" name="tGND_GNDA" color="7" fill="9" visible="yes" active="no"/>
+<layer number="54" name="bGND_GNDA" color="1" fill="9" visible="yes" active="no"/>
+<layer number="56" name="wert" color="7" fill="1" visible="yes" active="no"/>
+<layer number="57" name="tCAD" color="7" fill="1" visible="yes" active="no"/>
 <layer number="91" name="Nets" color="2" fill="1" visible="yes" active="yes"/>
 <layer number="92" name="Busses" color="1" fill="1" visible="yes" active="yes"/>
@@
 <part name="U$5" library="SparkFun-Aesthetics" deviceset="VIN" device=""/>
 <part name="C_M1" library="rcl" deviceset="C-US" device="C0402" value="0.1uF"/>
-<part name="JP1" library="SparkFun-Connectors" deviceset="M01" device="SMD-4.5X1.5" value="M01SMD-4.5X1.5"/>
-<part name="JP2" library="SparkFun-Connectors" deviceset="M01" device="SMD-4.5X1.5" value="M01SMD-4.5X1.5"/>
 <part name="C_3V2" library="rcl" deviceset="C-US" device="C0603" value="2.2uF"/>
 <part name="C_M2" library="rcl" deviceset="C-US" device="C0402" value="0.1uF"/>
@@
 <part name="P+9" library="SparkFun-Aesthetics" deviceset="3.3V" device=""/>
 <part name="U$11" library="SparkFun-Aesthetics" deviceset="VIN" device=""/>
-<part name="JP3" library="SparkFun-Connectors" deviceset="M01" device="SMD-4.5X1.5" value="M01SMD-4.5X1.5"/>
-<part name="JP4" library="SparkFun-Connectors" deviceset="M01" device="SMD-4.5X1.5" value="M01SMD-4.5X1.5"/>
 <part name="&lt;HEADER&gt;1" library="tekdemo" deviceset="M06X02" device="2MM_SMT"/>
 <part name="C1" library="SparkFun-Passives" deviceset="CAP_POL" device="PTH2"/>
@@
 <part name="R_P" library="SparkFun-Passives" deviceset="RESISTOR-ARRAY" device="0603-ARV" value="1k-10k"/>
 <part name="P+10" library="SparkFun-Aesthetics" deviceset="3.3V" device=""/>
+<part name="JP5" library="SparkFun-Connectors" deviceset="M01" device="SMD-4.5X1.5" value="M01SMD-4.5X1.5"/>
+<part name="JP6" library="SparkFun-Connectors" deviceset="M01" device="SMD-4.5X1.5" value="M01SMD-4.5X1.5"/>
+<part name="JP1" library="SparkFun-Connectors" deviceset="M01" device="SMD-4.5X1.5" value="M01SMD-4.5X1.5"/>
+<part name="JP3" library="SparkFun-Connectors" deviceset="M01" device="SMD-4.5X1.5" value="M01SMD-4.5X1.5"/>
 </parts>
 <sheets>
@@
 <instance part="U$5" gate="G$1" x="254" y="116.84" rot="R90"/>
 <instance part="C_M1" gate="G$1" x="220.98" y="35.56"/>
-<instance part="JP1" gate="G$1" x="261.62" y="45.72" rot="R270"/>
-<instance part="JP2" gate="G$1" x="261.62" y="22.86" rot="R90"/>
 <instance part="C_3V2" gate="G$1" x="114.3" y="198.12"/>
 <instance part="C_M2" gate="G$1" x="228.6" y="35.56"/>
@@
 <instance part="P+9" gate="G$1" x="160.02" y="157.48" rot="R90"/>
 <instance part="U$11" gate="G$1" x="157.48" y="154.94" rot="R90"/>
-<instance part="JP3" gate="G$1" x="274.32" y="45.72" rot="R270"/>
-<instance part="JP4" gate="G$1" x="274.32" y="22.86" rot="R90"/>
 <instance part="&lt;HEADER&gt;1" gate="G$1" x="205.74" y="213.36"/>
 <instance part="C1" gate="G$1" x="27.94" y="210.82"/>
@@
 <instance part="R_P" gate="B" x="215.9" y="127" rot="R90"/>
 <instance part="P+10" gate="G$1" x="215.9" y="147.32"/>
+<instance part="JP5" gate="G$1" x="261.62" y="58.42" rot="R270"/>
+<instance part="JP6" gate="G$1" x="274.32" y="58.42" rot="R270"/>
+<instance part="JP1" gate="G$1" x="261.62" y="15.24" rot="R90"/>
+<instance part="JP3" gate="G$1" x="274.32" y="15.24" rot="R90"/>
 </instances>
 <busses>
@@
 <wire x1="220.98" y1="38.1" x2="228.6" y2="38.1" width="0.1524" layer="91"/>
 <junction x="220.98" y="38.1"/>
-<pinref part="JP1" gate="G$1" pin="1"/>
 <pinref part="C_M2" gate="G$1" pin="1"/>
 <wire x1="228.6" y1="38.1" x2="236.22" y2="38.1" width="0.1524" layer="91"/>
 <junction x="228.6" y="38.1"/>
 <pinref part="C_M" gate="G$1" pin="1"/>
-<wire x1="236.22" y1="38.1" x2="261.62" y2="38.1" width="0.1524" layer="91"/>
+<wire x1="236.22" y1="38.1" x2="274.32" y2="38.1" width="0.1524" layer="91"/>
 <junction x="236.22" y="38.1"/>
-<pinref part="JP3" gate="G$1" pin="1"/>
-<wire x1="261.62" y1="38.1" x2="274.32" y2="38.1" width="0.1524" layer="91"/>
-<junction x="261.62" y="38.1"/>
 </segment>
 </net>
@@
 <wire x1="220.98" y1="30.48" x2="228.6" y2="30.48" width="0.1524" layer="91"/>
 <junction x="220.98" y="30.48"/>
-<pinref part="JP2" gate="G$1" pin="1"/>
 <pinref part="C_M2" gate="G$1" pin="2"/>
 <wire x1="228.6" y1="30.48" x2="236.22" y2="30.48" width="0.1524" layer="91"/>
 <junction x="228.6" y="30.48"/>
 <pinref part="C_M" gate="G$1" pin="2"/>
-<wire x1="236.22" y1="30.48" x2="261.62" y2="30.48" width="0.1524" layer="91"/>
+<wire x1="236.22" y1="30.48" x2="274.32" y2="30.48" width="0.1524" layer="91"/>
 <junction x="236.22" y="30.48"/>
-<pinref part="JP4" gate="G$1" pin="1"/>
-<wire x1="261.62" y1="30.48" x2="274.32" y2="30.48" width="0.1524" layer="91"/>
-<junction x="261.62" y="30.48"/>
-</segment>
-</net>
+</segment>
+</net>

Commit message: Added header routing and silkscreen
Parts:
- renumbered C_3V2 to C.3V, C_AV to C.AV, C_MAG to C.MAG, C_MOS to C.MOS, C_UC to C.UC, D_AV to D.AV, IC_V to IC.V, R_AV to R.AV, R_L to R.L, R_L1 to R.L1, R_L2 to R.L2, R_P to R.PU, R_PDA to R.PDA, R_PDB to R.PDB
Connections:
- removed net A6: UC.ADC6
- removed net PD3: UC.PD3(INT1)
- new net A6_HEADER_ADC: <HEADER>1.P$10, UC.ADC6
- new net PD2_HEADER_HW_INT: <HEADER>1.P$2, UC.PD2(INT0)
- net 3.3V: now also <HEADER>1.P$7
- net AS5050_INT: now also UC.PD3(INT1); no longer UC.PD2(INT0)
- net MISO: now also <HEADER>1.P$3
- net MOSI: now also <HEADER>1.P$8
- net M_GND: now also <HEADER>1.P$9
- net PD7: now also <HEADER>1.P$12
- net RESET: now also <HEADER>1.P$1
- net SCK: now also <HEADER>1.P$5
- net SCL/TX0: now also <HEADER>1.P$4
- net SDA/RXI: now also <HEADER>1.P$6
- net VIN: now also <HEADER>1.P$11

Commit message: Routed Headers, added header pinout in silk
Parts:
- renumbered <HEADER>1 to <HEADER>
Changed lines of the file:
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@@
 <part name="P+9" library="SparkFun-Aesthetics" deviceset="3.3V" device=""/>
 <part name="U$11" library="SparkFun-Aesthetics" deviceset="VIN" device=""/>
-<part name="&lt;HEADER&gt;1" library="tekdemo" deviceset="M06X02" device="2MM_SMT"/>
+<part name="&lt;HEADER&gt;" library="tekdemo" deviceset="M06X02" device="2MM_SMT"/>
 <part name="C1" library="SparkFun-Passives" deviceset="CAP_POL" device="PTH2"/>
 <part name="C2" library="SparkFun-Passives" deviceset="CAP_POL" device="C"/>
@@
 <instance part="P+9" gate="G$1" x="160.02" y="157.48" rot="R90"/>
 <instance part="U$11" gate="G$1" x="157.48" y="154.94" rot="R90"/>
-<instance part="&lt;HEADER&gt;1" gate="G$1" x="205.74" y="172.72"/>
+<instance part="&lt;HEADER&gt;" gate="G$1" x="205.74" y="172.72"/>
 <instance part="C1" gate="G$1" x="27.94" y="210.82"/>
 <instance part="C2" gate="G$1" x="35.56" y="210.82"/>
@@
 <wire x1="193.04" y1="185.42" x2="182.88" y2="185.42" width="0.1524" layer="91"/>
 <label x="182.88" y="185.42" size="1.778" layer="95"/>
-<pinref part="&lt;HEADER&gt;1" gate="G$1" pin="P$1"/>
+<pinref part="&lt;HEADER&gt;" gate="G$1" pin="P$1"/>
 </segment>
 </net>
@@
 <wire x1="193.04" y1="160.02" x2="182.88" y2="160.02" width="0.1524" layer="91"/>
 <label x="182.88" y="160.02" size="1.778" layer="95"/>
-<pinref part="&lt;HEADER&gt;1" gate="G$1" pin="P$11"/>
+<pinref part="&lt;HEADER&gt;" gate="G$1" pin="P$11"/>
 </segment>
 </net>
@@
 <wire x1="220.98" y1="165.1" x2="233.68" y2="165.1" width="0.1524" layer="91"/>
 <label x="228.6" y="165.1" size="1.778" layer="95"/>
-<pinref part="&lt;HEADER&gt;1" gate="G$1" pin="P$10"/>
+<pinref part="&lt;HEADER&gt;" gate="G$1" pin="P$10"/>
 </segment>
 </net>
@@
 <wire x1="220.98" y1="160.02" x2="236.22" y2="160.02" width="0.1524" layer="91"/>
 <label x="228.6" y="160.02" size="1.778" layer="95"/>
-<pinref part="&lt;HEADER&gt;1" gate="G$1" pin="P$12"/>
+<pinref part="&lt;HEADER&gt;" gate="G$1" pin="P$12"/>
 </segment>
 </net>
@@
 <wire x1="193.04" y1="175.26" x2="182.88" y2="175.26" width="0.1524" layer="91"/>
 <label x="182.88" y="175.26" size="1.778" layer="95"/>
-<pinref part="&lt;HEADER&gt;1" gate="G$1" pin="P$5"/>
+<pinref part="&lt;HEADER&gt;" gate="G$1" pin="P$5"/>
 </segment>
 </net>
@@
 <wire x1="193.04" y1="180.34" x2="182.88" y2="180.34" width="0.1524" layer="91"/>
 <label x="182.88" y="180.34" size="1.778" layer="95"/>
-<pinref part="&lt;HEADER&gt;1" gate="G$1" pin="P$3"/>
+<pinref part="&lt;HEADER&gt;" gate="G$1" pin="P$3"/>
 </segment>
 </net>
@@
 <wire x1="220.98" y1="170.18" x2="238.76" y2="170.18" width="0.1524" layer="91"/>
 <label x="226.06" y="170.18" size="1.778" layer="95"/>
-<pinref part="&lt;HEADER&gt;1" gate="G$1" pin="P$8"/>
+<pinref part="&lt;HEADER&gt;" gate="G$1" pin="P$8"/>
 </segment>
 </net>
@@
 <wire x1="193.04" y1="170.18" x2="182.88" y2="170.18" width="0.1524" layer="91"/>
 <label x="182.88" y="170.18" size="1.778" layer="95"/>
-<pinref part="&lt;HEADER&gt;1" gate="G$1" pin="P$7"/>
+<pinref part="&lt;HEADER&gt;" gate="G$1" pin="P$7"/>
 </segment>
 <segment>
@@
 <segment>
 <wire x1="193.04" y1="165.1" x2="182.88" y2="165.1" width="0.1524" layer="91"/>
-<pinref part="&lt;HEADER&gt;1" gate="G$1" pin="P$9"/>
+<pinref part="&lt;HEADER&gt;" gate="G$1" pin="P$9"/>
 <label x="182.88" y="165.1" size="1.778" layer="95"/>
 </segment>
@@
 <wire x1="220.98" y1="175.26" x2="231.14" y2="175.26" width="0.1524" layer="91"/>
 <label x="226.06" y="175.26" size="1.778" layer="95"/>
-<pinref part="&lt;HEADER&gt;1" gate="G$1" pin="P$6"/>
+<pinref part="&lt;HEADER&gt;" gate="G$1" pin="P$6"/>
 </segment>
 <segment>
@@
 <wire x1="220.98" y1="180.34" x2="233.68" y2="180.34" width="0.1524" layer="91"/>
 <label x="228.6" y="180.34" size="1.778" layer="95"/>
-<pinref part="&lt;HEADER&gt;1" gate="G$1" pin="P$4"/>
+<pinref part="&lt;HEADER&gt;" gate="G$1" pin="P$4"/>
 </segment>
 </net>
@@
 <wire x1="220.98" y1="185.42" x2="228.6" y2="185.42" width="0.1524" layer="91"/>
 <label x="223.52" y="185.42" size="1.778" layer="95"/>
-<pinref part="&lt;HEADER&gt;1" gate="G$1" pin="P$2"/>
-</segment>
-</net>
+<pinref part="&lt;HEADER&gt;" gate="G$1" pin="P$2"/>
+</segment>
+</net>

Commit message: verified functionality of board, added notes
Other:
- note added: "MAKE THESE PULL UPS INSTEAD OF PULL DOWN"
Changed lines of the file:
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@@
 during suspended/
 low-power modes</text>
+<text x="154.94" y="2.54" size="1.778" layer="91">MAKE THESE PULL UPS INSTEAD OF PULL DOWN</text>
 </plain>
 <instances>
